File: LSR_GPS_Tracker_Base_Station.brd (EAGLE design)
At the start: 78 x 83 mm, 36 parts, among them CON1 XT30PW-M

Commit message: Add files via upload
Parts:
- added U$4: GPS_ATGM336H_MOD, LSR_Modules:GPS_ATGM336H_FP
- LED1, LED2, LED3: value (none) -> LED; device adafruit:CHIPLED_0805 -> LSR_Generic_Parts:0805_LED
- RF1: value E22_900T22DC_MOD -> E22_900T22D_MOD; device LSR_Modules:E22_900T22DC_MOD_FP -> LSR_RF_WIFI:E22_900T22D_MOD_FP
- moved U$3 33.0 mm to (10.2, 47.0)
- moved R17 5.77 mm to (-7.62, 71.1)
- moved R15 5.38 mm to (-8.00, 81.0)
- moved R16 5.38 mm to (-8.00, 76.0)
- moved LED3 5.17 mm to (-13.1, 81.0), turned to 180 degrees
- moved LED1 4.99 mm to (-12.9, 76.0), turned to 180 degrees
- moved LED2 4.83 mm to (-12.7, 71.1), turned to 180 degrees
- moved GPS1 0.34 mm to (11.0, 42.2)
Connections:
- net VBATT renamed V_BATT
- removed net 3V3: COMP1.VCC, GPS1.VCC, J1.4, J2.11, S1.3, S2.3, S3.3, S4.3, S5.3, U$1.VCC, U$3.3V3-1, U$3.3V3-3
- removed net N$3: J1.10, U$3.18-A4/SDA0/PWM18
- removed net N$54: LED2.C, R17.1
- removed net N$55: LED3.C, R15.1
- new net 3.3V: COMP1.VCC, GPS1.VCC, J1.4, J2.11, S1.3, S2.3, S3.3, S4.3, S5.3, U$1.VCC, U$3.3V3-1, U$3.3V3-3, U$4.VCC
- new net GPS_PPS: J1.10, U$3.18-A4/SDA0/PWM18, U$4.PPS
- new net N$28: J2.22, U$3.2-OUT2/PWM02
- new net N$32: LED3.A, R15.2
- new net N$53: LED2.A, R17.2
- net 5V: now also R15.1; no longer LED3.A
- net GND: now also LED1.C, LED2.C, LED3.C, S6.1, U$4.GND; no longer R15.2, R16.2, R17.2
- net GPS_RX: now also U$4.RX
- net GPX_TX: now also U$4.TX
- net LED1: now also R16.1; no longer LED1.A
- net LED2: now also R17.1; no longer LED2.A
- net N$33: now also LED1.A, R16.2; no longer LED1.C, R16.1
- net PSU_EN: no longer J2.22, U$3.2-OUT2/PWM02
Routing:
- net 3.3V: track 0.00 -> 166.8 mm, vias 0 -> 2
- net 3V3: track 165.6 -> 0.00 mm, vias 2 -> 0
- net GPS_PPS: track 0.00 -> 18.9 mm, vias 0 -> 2
- net GPS_RX: track 8.95 -> 23.5 mm
- net GPX_TX: track 14.2 -> 25.6 mm
- net GND: track 271.5 -> 276.4 mm, vias 145 -> 136
- net N$54: track 3.32 -> 0.00 mm
- net N$55: track 3.32 -> 0.00 mm
- net N$53: track 0.00 -> 2.96 mm
- net N$32: track 0.00 -> 2.91 mm
- net PSU_EN: track 2.58 -> 0.00 mm
- net N$4: track 2.54 -> 0.00 mm
- net N$3: track 2.54 -> 0.00 mm
- net N$28: track 0.00 -> 2.54 mm
- net N$33: track 3.41 -> 2.73 mm
