File: LSR_GPS_Tracker_Base_Station.sch (EAGLE design)
At the start: 34 parts, among them CON1 XT30PW-M

Commit message: Add files via upload
Parts:
- added U$4: GPS_ATGM336H_MOD, LSR_Modules:GPS_ATGM336H_MOD
- LED1, LED2, LED3: value (none) -> LED; device adafruit:LEDCHIPLED_0805 -> LSR_Generic_Parts:LED
- RF1: value E22_900T22DC_MOD -> E22_900T22D_MOD; device LSR_Modules:E22_900T22DC_MOD -> LSR_RF_WIFI:E22_900T22D_MOD
Connections:
- net VBATT renamed V_BATT
- removed net 3V3: COMP1.VCC, GPS1.VCC, J1.4, J2.11, S1.2, S2.2, S3.2, S4.2, S5.2, U$1.VCC, U$3.3V3@1, U$3.3V3@2
- removed net N$3: J1.10, U$3.18-A4/SDA0/PWM18
- removed net N$54: LED2.C, R17.1
- removed net N$55: LED3.C, R15.1
- new net 3.3V: COMP1.VCC, GPS1.VCC, J1.4, J2.11, S1.2, S2.2, S3.2, S4.2, S5.2, U$1.VCC, U$3.3V3@1, U$3.3V3@2, U$4.VIN
- new net GPS_PPS: J1.10, U$3.18-A4/SDA0/PWM18, U$4.PPS
- new net N$28: J2.22, U$3.2-OUT2/PWM02
- new net N$32: LED3.A, R15.2
- new net N$53: LED2.A, R17.2
- net 5V: now also R15.1, U$3.VIN_5V; no longer LED3.A, U$3.VIN
- net GND: now also LED1.C, LED2.C, LED3.C, S6.1, U$4.GND; no longer R15.2, R16.2, R17.2
- net GPS_RX: now also U$4.RX
- net GPX_TX: now also U$4.TX
- net LED1: now also R16.1; no longer LED1.A
- net LED2: now also R17.1; no longer LED2.A
- net N$33: now also LED1.A, R16.2; no longer LED1.C, R16.1
- net PSU_EN: no longer J2.22, U$3.2-OUT2/PWM02
Other:
- note added: "<Notes>"
- note added: "Note: Reverse polarity protection TSM2323CX MOSFET P-CH 20V 4.7A SOT23 RDS: 39mOhm @ 4.7A, 4.5V (Option 2: SI2369BDS-T1-GE3) Note: Resettable 1812 Fuse Hold: 2A Trip: 3.5A Max: 12V, 100A"
- moved on the sheet: F1, J1, J2, PS1, R10, R11, R15, R16, R17, R7, R8, R9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
